File: PWR_Supply/DC.sch (KiCad schematic (older format))
At the start: 1 part, among them J6 

Commit message: Izlabots Majas Darbs Nr.2
Parts:
- removed J6: (no value), symbol Connector_Generic:Conn_01x05
- added J2: (no value), symbol Connector_Generic:Conn_01x05
Connections:
- net GND: now also J2.5 (Pin_5)
- new net +12V: J2.4 (Pin_4)
- new net +3V3: J2.1 (Pin_1)
- new net +5V: J2.2 (Pin_2)
- new net +9V: J2.3 (Pin_3)
Changed lines of the file:
@@
 EESchema Schematic File Version 4
-LIBS:PWR_Supply-cache
 EELAYER 26 0
 EELAYER END
@@
 Comment4 ""
 $EndDescr
+Text HLabel 5250 3750 0    50   Input ~ 0
++5
+Text HLabel 5250 3600 0    50   Input ~ 0
++3.3
+Text HLabel 5250 3900 0    50   Input ~ 0
++9
+Text HLabel 5250 4050 0    50   Input ~ 0
++12
+Text HLabel 5250 4200 0    50   Input ~ 0
+GND
+Wire Wire Line
+	5250 4200 5350 4200
+Wire Wire Line
+	5250 3600 5350 3600
+Wire Wire Line
+	5250 3750 5350 3750
+Wire Wire Line
+	5250 4050 5350 4050
 $Comp
-L Connector_Generic:Conn_01x05 J6
-U 1 1 5C85B429
+L power:+3.3V #PWR0110
+U 1 1 5C909660
+P 5350 3600
+F 0 "#PWR0110" H 5350 3450 50  0001 C CNN
+F 1 "+3.3V" H 5250 3700 39  0000 C CNN
+F 2 "" H 5350 3600 50  0001 C CNN
+F 3 "" H 5350 3600 50  0001 C CNN
+	1    5350 3600
+	1    0    0    -1
+$EndComp
+Connection ~ 5350 3600
+Wire Wire Line
+	5350 3600 5450 3600
+$Comp
+L Connector_Generic:Conn_01x05 J2
+U 1 1 5C909712
 P 5650 3900
-F 0 "J6" H 5729 3942 50  0000 L CNN
-F 1 "  " H 5729 3851 50  0000 L CNN
+F 0 "J2" H 5730 3942 50  0000 L CNN
+F 1 " " H 5730 3851 50  0000 L CNN
 F 2 "" H 5650 3900 50  0001 C CNN
 F 3 "~" H 5650 3900 50  0001 C CNN
@@
 	1    0    0    -1
 $EndComp
-Text HLabel 5250 3800 0    50   Input ~ 0
-+5
-Text HLabel 5250 3700 0    50   Input ~ 0
-+3.3
-Text HLabel 5250 3900 0    50   Input ~ 0
-+9
-Text HLabel 5250 4000 0    50   Input ~ 0
-+12
-Text HLabel 5250 4100 0    50   Input ~ 0
-GND
 $Comp
-L power:PWR_FLAG #FLG0109
-U 1 1 5C8E4AF3
-P 5350 3700
-F 0 "#FLG0109" H 5350 3775 50  0001 C CNN
-F 1 "PWR_FLAG" H 4650 3700 50  0000 C CNN
-F 2 "" H 5350 3700 50  0001 C CNN
-F 3 "~" H 5350 3700 50  0001 C CNN
-	1    5350 3700
+L power:+9V #PWR0111
+U 1 1 5C90975E
+P 5350 3900
+F 0 "#PWR0111" H 5350 3750 50  0001 C CNN
+F 1 "+9V" H 5250 3950 39  0000 C CNN
+F 2 "" H 5350 3900 50  0001 C CNN
+F 3 "" H 5350 3900 50  0001 C CNN
+	1    5350 3900
 	1    0    0    -1
 $EndComp
 Wire Wire Line
-	5350 3700 5450 3700
+	5250 3900 5350 3900
+Connection ~ 5350 3900
+Wire Wire Line
+	5350 3900 5450 3900
 $Comp
-L power:PWR_FLAG #FLG0110
-U 1 1 5C8E537F
-P 5400 3800
-F 0 "#FLG0110" H 5400 3875 50  0001 C CNN
-F 1 "PWR_FLAG" H 4650 3800 50  0000 C CNN
-F 2 "" H 5400 3800 50  0001 C CNN
-F 3 "~" H 5400 3800 50  0001 C CNN
-	1    5400 3800
+L power:+5V #PWR0112
+U 1 1 5C909A21
+P 5350 3750
+F 0 "#PWR0112" H 5350 3600 50  0001 C CNN
+F 1 "+5V" H 5250 3800 39  0000 C CNN
+F 2 "" H 5350 3750 50  0001 C CNN
+F 3 "" H 5350 3750 50  0001 C CNN
+	1    5350 3750
 	1    0    0    -1
 $EndComp
+Connection ~ 5350 3750
 Wire Wire Line
-	5400 3800 5450 3800
+	5350 3750 5450 3750
 $Comp
-L power:PWR_FLAG #FLG0111
-U 1 1 5C8E538E
-P 5350 3900
-F 0 "#FLG0111" H 5350 3975 50  0001 C CNN
-F 1 "PWR_FLAG" H 4650 3900 50  0000 C CNN
-F 2 "" H 5350 3900 50  0001 C CNN
-F 3 "~" H 5350 3900 50  0001 C CNN
-	1    5350 3900
+L power:+12V #PWR0113
+U 1 1 5C909AF7
+P 5350 4050
+F 0 "#PWR0113" H 5350 3900 50  0001 C CNN
+F 1 "+12V" H 5200 4100 39  0000 C CNN
+F 2 "" H 5350 4050 50  0001 C CNN
+F 3 "" H 5350 4050 50  0001 C CNN
+	1    5350 4050
 	1    0    0    -1
 $EndComp
+Connection ~ 5350 4050
+Wire Wire Line
+	5350 4050 5450 4050
 $Comp
-L power:PWR_FLAG #FLG0112
-U 1 1 5C8E539D
-P 5400 4000
-F 0 "#FLG0112" H 5400 4075 50  0001 C CNN
-F 1 "PWR_FLAG" H 4650 4000 50  0000 C CNN
-F 2 "" H 5400 4000 50  0001 C CNN
-F 3 "~" H 5400 4000 50  0001 C CNN
-	1    5400 4000
+L power:GND #PWR0114
+U 1 1 5C909B62
+P 5350 4200
+F 0 "#PWR0114" H 5350 3950 50  0001 C CNN
+F 1 "GND" H 5355 4027 50  0000 C CNN
+F 2 "" H 5350 4200 50  0001 C CNN
+F 3 "" H 5350 4200 50  0001 C CNN
+	1    5350 4200
 	1    0    0    -1
 $EndComp
-$Comp
-L power:PWR_FLAG #FLG0113
-U 1 1 5C8E53D1
-P 5350 4100
-F 0 "#FLG0113" H 5350 4175 50  0001 C CNN
-F 1 "PWR_FLAG" H 4650 4100 50  0000 C CNN
-F 2 "" H 5350 4100 50  0001 C CNN
-F 3 "~" H 5350 4100 50  0001 C CNN
-	1    5350 4100
-	1    0    0    -1
-$EndComp
+Connection ~ 5350 4200
 Wire Wire Line
-	5350 3900 5450 3900
+	5350 4200 5450 4200
 Wire Wire Line
-	5400 4000 5450 4000
+	5450 3700 5450 3600
 Wire Wire Line
-	5350 4100 5450 4100
-Connection ~ 5350 3700
+	5450 3800 5450 3750
 Wire Wire Line
-	5250 3700 5350 3700
-Connection ~ 5400 3800
+	5450 4050 5450 4000
 Wire Wire Line
-	5250 3800 5400 3800
-Connection ~ 5350 3900
-Wire Wire Line
-	5250 3900 5350 3900
-Connection ~ 5400 4000
-Wire Wire Line
-	5250 4000 5400 4000
-Connection ~ 5350 4100
-Wire Wire Line
-	5250 4100 5350 4100
+	5450 4200 5450 4100
 $EndSCHEMATC
