File: PWR_Supply/PWR_Supply.sch (KiCad schematic (older format))
At the start: 0 parts

Commit message: Izlabots Majas Darbs Nr.2
Connections:
- wire segments 29 -> 23
Changed lines of the file:
@@
 EESchema Schematic File Version 4
-LIBS:PWR_Supply-cache
 EELAYER 26 0
 EELAYER END
@@
 F4 "+12" I R 3450 6950 50
 $EndSheet
-Text GLabel 3700 3000 2    50   Input ~ 0
+Text GLabel 3700 2950 2    50   Input ~ 0
 BUS
-Wire Wire Line
-	3450 1400 3650 1400
-Wire Wire Line
-	3650 1400 3700 1350
-Wire Wire Line
-	3450 1650 3650 1650
-Wire Wire Line
-	3650 1650 3700 1600
-Wire Bus Line
-	3700 1600 3700 1250
-Text GLabel 3700 1250 2    50   Input ~ 0
+Text GLabel 3700 1200 2    50   Input ~ 0
 BUS
-Wire Wire Line
-	8950 1800 9150 1800
-Wire Wire Line
-	9150 1800 9200 1750
-Wire Wire Line
-	8950 2000 9150 2000
-Wire Wire Line
-	9150 2000 9200 1950
-Wire Bus Line
-	9200 1950 9200 1650
-Text GLabel 9200 1650 2    50   Input ~ 0
+Text GLabel 9150 1600 2    50   Input ~ 0
 BUS
-Wire Wire Line
-	3450 3150 3650 3150
-Wire Wire Line
-	3650 3150 3700 3100
-Wire Wire Line
-	3450 3400 3650 3400
-Wire Wire Line
-	3650 3400 3700 3350
-Wire Bus Line
-	3700 3350 3700 3000
-Wire Wire Line
-	3450 4700 3650 4700
-Wire Wire Line
-	3650 4700 3700 4650
-Wire Wire Line
-	3450 4900 3650 4900
-Wire Wire Line
-	3650 4900 3700 4850
-Wire Bus Line
-	3700 4850 3700 4550
-Text GLabel 3700 4550 2    50   Input ~ 0
+Text GLabel 3650 4500 2    50   Input ~ 0
 BUS
 $Sheet
@@
 F6 "GND" I L 5800 3800 50
 $EndSheet
-Text GLabel 5700 3150 0    50   Input ~ 0
+Text GLabel 5550 3150 0    50   Input ~ 0
 DC
-Wire Wire Line
-	3650 6650 3700 6600
-Wire Wire Line
-	3450 6650 3650 6650
-Wire Wire Line
-	3450 6450 3650 6450
-Wire Wire Line
-	3650 6450 3700 6400
-Text GLabel 3700 6300 2    50   Input ~ 0
+Text GLabel 3650 6250 2    50   Input ~ 0
 BUS
-Wire Bus Line
-	3700 6600 3700 6300
 Text GLabel 5650 3800 0    50   Input ~ 0
 BUS
 Wire Wire Line
 	5650 3800 5800 3800
-Entry Bus Bus
-	5700 3300 5800 3400
-Entry Bus Bus
-	5700 3400 5800 3500
-Entry Bus Bus
-	5700 3500 5800 3600
-Entry Bus Bus
-	5700 3600 5800 3700
 Entry Wire Line
 	4200 950  4300 850
@@
 Entry Wire Line
 	4500 950  4600 850
-Entry Wire Line
-	4650 950  4750 850
 Text GLabel 4100 850  1    50   Input ~ 0
 DC
@@
 Wire Wire Line
 	3450 5250 4500 5250
-Wire Bus Line
-	5700 3150 5700 3650
-Wire Bus Line
-	4100 850  5000 850
 $Sheet
 S 5650 900  3300 1900
@@
 F3 "VCC" I R 8950 1800 50
 $EndSheet
+Entry Wire Line
+	5550 3300 5650 3400
+Entry Wire Line
+	5550 3400 5650 3500
+Entry Wire Line
+	5550 3500 5650 3600
+Entry Wire Line
+	3550 4700 3650 4600
+Entry Wire Line
+	3550 4900 3650 4800
+Entry Wire Line
+	3550 6650 3650 6550
+Entry Wire Line
+	3550 6450 3650 6350
+Entry Wire Line
+	3600 1650 3700 1550
+Entry Wire Line
+	3600 1400 3700 1300
+Entry Wire Line
+	9050 1800 9150 1700
+Entry Wire Line
+	9050 2000 9150 1900
+Entry Wire Line
+	4650 950  4750 850
+Wire Wire Line
+	3450 1400 3600 1400
+Wire Wire Line
+	3450 1650 3600 1650
+Wire Wire Line
+	3450 3150 3600 3150
+Wire Wire Line
+	3450 3400 3600 3400
+Wire Wire Line
+	3450 4700 3550 4700
+Wire Wire Line
+	3450 4900 3550 4900
+Wire Wire Line
+	3450 6450 3550 6450
+Wire Wire Line
+	3450 6650 3550 6650
+Wire Wire Line
+	8950 1800 9050 1800
+Wire Wire Line
+	8950 2000 9050 2000
+Wire Wire Line
+	5800 3400 5650 3400
+Wire Wire Line
+	5650 3500 5800 3500
+Wire Wire Line
+	5650 3600 5800 3600
+Entry Wire Line
+	5550 3600 5650 3700
+Wire Wire Line
+	5650 3700 5800 3700
+Entry Wire Line
+	3600 3400 3700 3300
+Entry Wire Line
+	3600 3150 3700 3050
+Wire Bus Line
+	3700 2950 3700 3300
+Wire Bus Line
+	3650 4500 3650 4800
+Wire Bus Line
+	3650 6250 3650 6550
+Wire Bus Line
+	9150 1600 9150 1900
+Wire Bus Line
+	3700 1200 3700 1550
+Wire Bus Line
+	4100 850  5000 850
+Wire Bus Line
+	5550 3150 5550 3650
 $EndSCHEMATC
