File: PWR_Supply/12V_DC.sch (KiCad schematic (older format))
At the start: 3 parts, among them U4 L7812

Commit message: Izlabots Majas Darbs Nr.2
Connections:
- net +12 renamed +12V
Changed lines of the file:
@@
 EESchema Schematic File Version 4
-LIBS:PWR_Supply-cache
 EELAYER 26 0
 EELAYER END
@@
 Wire Wire Line
 	5550 3400 6150 3400
-Wire Wire Line
-	5000 3000 4750 3000
 Connection ~ 5000 3000
 Connection ~ 5000 3400
@@
 Text HLabel 4550 3400 0    50   Input ~ 0
 GND
-$Comp
-L power:PWR_FLAG #FLG0107
-U 1 1 5C8E3D4C
-P 4750 3500
-F 0 "#FLG0107" H 4750 3575 50  0001 C CNN
-F 1 "PWR_FLAG" H 4750 3673 50  0000 C CNN
-F 2 "" H 4750 3500 50  0001 C CNN
-F 3 "~" H 4750 3500 50  0001 C CNN
-	1    4750 3500
-	-1   0    0    1
-$EndComp
-$Comp
-L power:PWR_FLAG #FLG0108
-U 1 1 5C8E3D64
-P 4750 2900
-F 0 "#FLG0108" H 4750 2975 50  0001 C CNN
-F 1 "PWR_FLAG" H 4750 3074 50  0000 C CNN
-F 2 "" H 4750 2900 50  0001 C CNN
-F 3 "~" H 4750 2900 50  0001 C CNN
-	1    4750 2900
-	1    0    0    -1
-$EndComp
 Wire Wire Line
-	4750 3000 4750 2900
-Connection ~ 4750 3000
-Wire Wire Line
-	4750 3000 4550 3000
-Wire Wire Line
-	4550 3400 4750 3400
-Wire Wire Line
-	4750 3500 4750 3400
-Connection ~ 4750 3400
-Wire Wire Line
-	4750 3400 5000 3400
-Wire Wire Line
-	6150 3000 6450 3000
+	6150 3000 6300 3000
 Connection ~ 6150 3000
 Text HLabel 6450 3000 2    50   Input ~ 0
 +12
+Wire Wire Line
+	4550 3000 4700 3000
+Wire Wire Line
+	4550 3400 4700 3400
+$Comp
+L power:VCC #PWR0107
+U 1 1 5C8D31E3
+P 4700 3000
+F 0 "#PWR0107" H 4700 2850 50  0001 C CNN
+F 1 "VCC" H 4717 3173 50  0000 C CNN
+F 2 "" H 4700 3000 50  0001 C CNN
+F 3 "" H 4700 3000 50  0001 C CNN
+	1    4700 3000
+	1    0    0    -1
+$EndComp
+Connection ~ 4700 3000
+Wire Wire Line
+	4700 3000 5000 3000
+$Comp
+L power:GND #PWR0108
+U 1 1 5C8D3214
+P 4700 3400
+F 0 "#PWR0108" H 4700 3150 50  0001 C CNN
+F 1 "GND" H 4705 3227 50  0000 C CNN
+F 2 "" H 4700 3400 50  0001 C CNN
+F 3 "" H 4700 3400 50  0001 C CNN
+	1    4700 3400
+	1    0    0    -1
+$EndComp
+Connection ~ 4700 3400
+Wire Wire Line
+	4700 3400 5000 3400
+$Comp
+L power:+12V #PWR0117
+U 1 1 5C909F4C
+P 6300 3000
+F 0 "#PWR0117" H 6300 2850 50  0001 C CNN
+F 1 "+12V" H 6315 3173 50  0000 C CNN
+F 2 "" H 6300 3000 50  0001 C CNN
+F 3 "" H 6300 3000 50  0001 C CNN
+	1    6300 3000
+	1    0    0    -1
+$EndComp
+Connection ~ 6300 3000
+Wire Wire Line
+	6300 3000 6450 3000
 $EndSCHEMATC

Commit message: Izlabots majas darbs Nr.2
Changed lines of the file:
@@
 EESchema Schematic File Version 4
+LIBS:PWR_Supply-cache
 EELAYER 26 0
 EELAYER END
@@
 Text HLabel 4550 3400 0    50   Input ~ 0
 GND
-Wire Wire Line
-	6150 3000 6300 3000
 Connection ~ 6150 3000
-Text HLabel 6450 3000 2    50   Input ~ 0
+Text HLabel 6450 3000 2    50   Output ~ 0
 +12
 Wire Wire Line
-	4550 3000 4700 3000
+	4700 3400 5000 3400
 Wire Wire Line
 	4550 3400 4700 3400
+Connection ~ 4700 3400
+$Comp
+L power:GND #PWR0108
+U 1 1 5C8D3214
+P 4700 3400
+F 0 "#PWR0108" H 4700 3150 50  0001 C CNN
+F 1 "GND" H 4705 3227 50  0000 C CNN
+F 2 "" H 4700 3400 50  0001 C CNN
+F 3 "" H 4700 3400 50  0001 C CNN
+	1    4700 3400
+	1    0    0    -1
+$EndComp
+Wire Wire Line
+	4700 3000 5000 3000
+Wire Wire Line
+	4550 3000 4700 3000
+Connection ~ 4700 3000
 $Comp
 L power:VCC #PWR0107
@@
 	1    0    0    -1
 $EndComp
-Connection ~ 4700 3000
 Wire Wire Line
-	4700 3000 5000 3000
-$Comp
-L power:GND #PWR0108
-U 1 1 5C8D3214
-P 4700 3400
-F 0 "#PWR0108" H 4700 3150 50  0001 C CNN
-F 1 "GND" H 4705 3227 50  0000 C CNN
-F 2 "" H 4700 3400 50  0001 C CNN
-F 3 "" H 4700 3400 50  0001 C CNN
-	1    4700 3400
-	1    0    0    -1
-$EndComp
-Connection ~ 4700 3400
+	6300 3000 6450 3000
 Wire Wire Line
-	4700 3400 5000 3400
+	6150 3000 6300 3000
+Connection ~ 6300 3000
 $Comp
 L power:+12V #PWR0117
@@
 	1    0    0    -1
 $EndComp
-Connection ~ 6300 3000
-Wire Wire Line
-	6300 3000 6450 3000
 $EndSCHEMATC

Commit message: Izlabots majas darbs Nr.2
Parts:
- U4: value L7812 -> LM7812
Changed lines of the file:
@@
 P 5550 3000
 F 0 "U4" H 5550 3242 50  0000 C CNN
-F 1 "L7812" H 5550 3151 50  0000 C CNN
+F 1 "LM7812" H 5550 3151 50  0000 C CNN
 F 2 "" H 5575 2850 50  0001 L CIN
-F 3 "http://www.st.com/content/ccc/resource/technical/document/datasheet/41/4f/b3/b0/12/d4/47/88/CD00000444.pdf/files/CD00000444.pdf/jcr:content/translations/en.CD00000444.pdf" H 5550 2950 50  0001 C CNN
+F 3 "https://pdf1.alldatasheet.com/datasheet-pdf/view/85508/ETC/LM7812.html" H 5550 2950 50  0001 C CNN
 	1    5550 3000
 	1    0    0    -1
