File: PWR_Supply/3.3V_DC.sch (KiCad schematic (older format))
At the start: 3 parts, among them U2 LD1117S33

Commit message: Izlabots Majas Darbs Nr.2
Connections:
- net +3.3 renamed +3V3
Changed lines of the file:
@@
 EESchema Schematic File Version 4
-LIBS:PWR_Supply-cache
 EELAYER 26 0
 EELAYER END
@@
 Text HLabel 4650 2950 0    50   Input ~ 0
 VCC
-Wire Wire Line
-	4650 3450 4800 3450
 Connection ~ 5100 2950
-Wire Wire Line
-	4650 2950 4800 2950
-$Comp
-L power:PWR_FLAG #FLG0101
-U 1 1 5C8E155C
-P 4800 2850
-F 0 "#FLG0101" H 4800 2925 50  0001 C CNN
-F 1 "PWR_FLAG" H 4800 3024 50  0000 C CNN
-F 2 "" H 4800 2850 50  0001 C CNN
-F 3 "~" H 4800 2850 50  0001 C CNN
-	1    4800 2850
-	1    0    0    -1
-$EndComp
-$Comp
-L power:PWR_FLAG #FLG0102
-U 1 1 5C8E17E5
-P 4800 3550
-F 0 "#FLG0102" H 4800 3625 50  0001 C CNN
-F 1 "PWR_FLAG" H 4800 3723 50  0000 C CNN
-F 2 "" H 4800 3550 50  0001 C CNN
-F 3 "~" H 4800 3550 50  0001 C CNN
-	1    4800 3550
-	-1   0    0    1
-$EndComp
-Wire Wire Line
-	4800 2950 4800 2850
-Connection ~ 4800 2950
-Wire Wire Line
-	4800 2950 5100 2950
-Wire Wire Line
-	4800 3550 4800 3450
-Connection ~ 4800 3450
-Wire Wire Line
-	4800 3450 5100 3450
 Text HLabel 6450 2950 2    50   Input ~ 0
 +3.3
 Connection ~ 6100 2950
 Wire Wire Line
-	6100 2950 6450 2950
+	6100 2950 6300 2950
 Wire Wire Line
 	5900 2950 6100 2950
+Wire Wire Line
+	4650 3450 4800 3450
+Wire Wire Line
+	4650 2950 4800 2950
+$Comp
+L power:VCC #PWR0101
+U 1 1 5C8D2B77
+P 4800 2800
+F 0 "#PWR0101" H 4800 2650 50  0001 C CNN
+F 1 "VCC" H 4817 2973 50  0000 C CNN
+F 2 "" H 4800 2800 50  0001 C CNN
+F 3 "" H 4800 2800 50  0001 C CNN
+	1    4800 2800
+	1    0    0    -1
+$EndComp
+Wire Wire Line
+	4800 2800 4800 2850
+Connection ~ 4800 2950
+Wire Wire Line
+	4800 2950 5100 2950
+$Comp
+L power:GND #PWR0102
+U 1 1 5C8D2C7F
+P 4800 3550
+F 0 "#PWR0102" H 4800 3300 50  0001 C CNN
+F 1 "GND" H 4805 3377 50  0000 C CNN
+F 2 "" H 4800 3550 50  0001 C CNN
+F 3 "" H 4800 3550 50  0001 C CNN
+	1    4800 3550
+	1    0    0    -1
+$EndComp
+Wire Wire Line
+	4800 3550 4800 3500
+Connection ~ 4800 3450
+Wire Wire Line
+	4800 3450 5100 3450
+$Comp
+L power:PWR_FLAG #FLG0101
+U 1 1 5C8D2EF8
+P 4800 3500
+F 0 "#FLG0101" H 4800 3575 50  0001 C CNN
+F 1 "PWR_FLAG" V 4800 3628 50  0000 L CNN
+F 2 "" H 4800 3500 50  0001 C CNN
+F 3 "~" H 4800 3500 50  0001 C CNN
+	1    4800 3500
+	0    1    1    0
+$EndComp
+Connection ~ 4800 3500
+Wire Wire Line
+	4800 3500 4800 3450
+$Comp
+L power:PWR_FLAG #FLG0102
+U 1 1 5C8D303E
+P 4800 2850
+F 0 "#FLG0102" H 4800 2925 50  0001 C CNN
+F 1 "PWR_FLAG" V 4800 2978 50  0000 L CNN
+F 2 "" H 4800 2850 50  0001 C CNN
+F 3 "~" H 4800 2850 50  0001 C CNN
+	1    4800 2850
+	0    1    1    0
+$EndComp
+Connection ~ 4800 2850
+Wire Wire Line
+	4800 2850 4800 2950
+$Comp
+L power:+3.3V #PWR0109
+U 1 1 5C90961E
+P 6300 2950
+F 0 "#PWR0109" H 6300 2800 50  0001 C CNN
+F 1 "+3.3V" H 6315 3123 50  0000 C CNN
+F 2 "" H 6300 2950 50  0001 C CNN
+F 3 "" H 6300 2950 50  0001 C CNN
+	1    6300 2950
+	1    0    0    -1
+$EndComp
+Connection ~ 6300 2950
+Wire Wire Line
+	6300 2950 6450 2950
 $EndSCHEMATC

Commit message: Izlabots majas darbs Nr.2
Changed lines of the file:
@@
 EESchema Schematic File Version 4
+LIBS:PWR_Supply-cache
 EELAYER 26 0
 EELAYER END
@@
 VCC
 Connection ~ 5100 2950
-Text HLabel 6450 2950 2    50   Input ~ 0
+Text HLabel 6450 2950 2    50   Output ~ 0
 +3.3
 Connection ~ 6100 2950
 Wire Wire Line
-	6100 2950 6300 2950
-Wire Wire Line
 	5900 2950 6100 2950
 Wire Wire Line
+	4800 3450 5100 3450
+Wire Wire Line
 	4650 3450 4800 3450
+Connection ~ 4800 3450
+Wire Wire Line
+	4800 3550 4800 3500
+Wire Wire Line
+	4800 3500 4800 3450
+Connection ~ 4800 3500
+$Comp
+L power:PWR_FLAG #FLG0101
+U 1 1 5C8D2EF8
+P 4800 3500
+F 0 "#FLG0101" H 4800 3575 50  0001 C CNN
+F 1 "PWR_FLAG" V 4800 3628 50  0000 L CNN
+F 2 "" H 4800 3500 50  0001 C CNN
+F 3 "~" H 4800 3500 50  0001 C CNN
+	1    4800 3500
+	0    1    1    0
+$EndComp
+$Comp
+L power:GND #PWR0102
+U 1 1 5C8D2C7F
+P 4800 3550
+F 0 "#PWR0102" H 4800 3300 50  0001 C CNN
+F 1 "GND" H 4805 3377 50  0000 C CNN
+F 2 "" H 4800 3550 50  0001 C CNN
+F 3 "" H 4800 3550 50  0001 C CNN
+	1    4800 3550
+	1    0    0    -1
+$EndComp
+$Comp
+L power:PWR_FLAG #FLG0102
+U 1 1 5C8D303E
+P 4800 2850
+F 0 "#FLG0102" H 4800 2925 50  0001 C CNN
+F 1 "PWR_FLAG" V 4800 2978 50  0000 L CNN
+F 2 "" H 4800 2850 50  0001 C CNN
+F 3 "~" H 4800 2850 50  0001 C CNN
+	1    4800 2850
+	0    1    1    0
+$EndComp
+Wire Wire Line
+	4800 2800 4800 2850
+Wire Wire Line
+	4800 2950 5100 2950
 Wire Wire Line
 	4650 2950 4800 2950
+Connection ~ 4800 2950
+Connection ~ 4800 2850
+Wire Wire Line
+	4800 2850 4800 2950
 $Comp
 L power:VCC #PWR0101
@@
 $EndComp
 Wire Wire Line
-	4800 2800 4800 2850
-Connection ~ 4800 2950
+	6300 2950 6450 2950
 Wire Wire Line
-	4800 2950 5100 2950
-$Comp
-L power:GND #PWR0102
-U 1 1 5C8D2C7F
-P 4800 3550
-F 0 "#PWR0102" H 4800 3300 50  0001 C CNN
-F 1 "GND" H 4805 3377 50  0000 C CNN
-F 2 "" H 4800 3550 50  0001 C CNN
-F 3 "" H 4800 3550 50  0001 C CNN
-	1    4800 3550
-	1    0    0    -1
-$EndComp
-Wire Wire Line
-	4800 3550 4800 3500
-Connection ~ 4800 3450
-Wire Wire Line
-	4800 3450 5100 3450
-$Comp
-L power:PWR_FLAG #FLG0101
-U 1 1 5C8D2EF8
-P 4800 3500
-F 0 "#FLG0101" H 4800 3575 50  0001 C CNN
-F 1 "PWR_FLAG" V 4800 3628 50  0000 L CNN
-F 2 "" H 4800 3500 50  0001 C CNN
-F 3 "~" H 4800 3500 50  0001 C CNN
-	1    4800 3500
-	0    1    1    0
-$EndComp
-Connection ~ 4800 3500
-Wire Wire Line
-	4800 3500 4800 3450
-$Comp
-L power:PWR_FLAG #FLG0102
-U 1 1 5C8D303E
-P 4800 2850
-F 0 "#FLG0102" H 4800 2925 50  0001 C CNN
-F 1 "PWR_FLAG" V 4800 2978 50  0000 L CNN
-F 2 "" H 4800 2850 50  0001 C CNN
-F 3 "~" H 4800 2850 50  0001 C CNN
-	1    4800 2850
-	0    1    1    0
-$EndComp
-Connection ~ 4800 2850
-Wire Wire Line
-	4800 2850 4800 2950
+	6100 2950 6300 2950
+Connection ~ 6300 2950
 $Comp
 L power:+3.3V #PWR0109
@@
 	1    0    0    -1
 $EndComp
-Connection ~ 6300 2950
-Wire Wire Line
-	6300 2950 6450 2950
 $EndSCHEMATC

Commit message: Izlabots majas darbs Nr.2
Parts:
- U2: value LD1117S33 -> LM7833
Changed lines of the file:
@@
 	5600 3450 6100 3450
 Connection ~ 5100 3450
-$Comp
-L Regulator_Linear:LD1117S33TR_SOT223 U2
-U 1 1 5C857F81
-P 5600 2950
-F 0 "U2" H 5600 3192 50  0000 C CNN
-F 1 "LD1117S33" H 5600 3101 50  0000 C CNN
-F 2 "Package_TO_SOT_SMD:SOT-223-3_TabPin2" H 5600 3150 50  0001 C CNN
-F 3 "http://www.st.com/st-web-ui/static/active/en/resource/technical/document/datasheet/CD00000544.pdf" H 5700 2700 50  0001 C CNN
-	1    5600 2950
-	1    0    0    -1
-$EndComp
 Text HLabel 4650 3450 0    50   Input ~ 0
 GND
@@
 	1    0    0    -1
 $EndComp
+$Comp
+L Regulator_Linear:LD1117S33TR_SOT223 U2
+U 1 1 5C857F81
+P 5600 2950
+F 0 "U2" H 5600 3192 50  0000 C CNN
+F 1 "LM7833" H 5600 3101 50  0000 C CNN
+F 2 "Package_TO_SOT_SMD:SOT-223-3_TabPin2" H 5600 3150 50  0001 C CNN
+F 3 "http://pdf1.alldatasheet.com/datasheet-pdf/view/237960/TAITRON/LM7833.html" H 5700 2700 50  0001 C CNN
+	1    5600 2950
+	1    0    0    -1
+$EndComp
