File: PWR_Supply/5V_DC.sch (KiCad schematic (older format))
At the start: 3 parts, among them U1 L7805

Commit message: Izlabots Majas Darbs Nr.2
Connections:
- net +5 renamed +5V
Changed lines of the file:
@@
 EESchema Schematic File Version 4
-LIBS:PWR_Supply-cache
 EELAYER 26 0
 EELAYER END
@@
 $EndComp
 Wire Wire Line
-	6050 3250 6350 3250
+	6050 3250 6250 3250
 Connection ~ 6050 3250
+Connection ~ 5000 3650
+Connection ~ 5000 3250
+Text HLabel 6350 3250 2    50   Input ~ 0
++5
+Wire Wire Line
+	4600 3250 4750 3250
 Wire Wire Line
 	4600 3650 4750 3650
-Connection ~ 5000 3650
 $Comp
-L power:PWR_FLAG #FLG0103
-U 1 1 5C8E322F
-P 4750 3150
-F 0 "#FLG0103" H 4750 3225 50  0001 C CNN
-F 1 "PWR_FLAG" H 4750 3324 50  0000 C CNN
-F 2 "" H 4750 3150 50  0001 C CNN
-F 3 "~" H 4750 3150 50  0001 C CNN
-	1    4750 3150
+L power:VCC #PWR0103
+U 1 1 5C8D30D8
+P 4750 3250
+F 0 "#PWR0103" H 4750 3100 50  0001 C CNN
+F 1 "VCC" H 4767 3423 50  0000 C CNN
+F 2 "" H 4750 3250 50  0001 C CNN
+F 3 "" H 4750 3250 50  0001 C CNN
+	1    4750 3250
 	1    0    0    -1
 $EndComp
+Connection ~ 4750 3250
+Wire Wire Line
+	4750 3250 5000 3250
 $Comp
-L power:PWR_FLAG #FLG0104
-U 1 1 5C8E3255
-P 4750 3750
-F 0 "#FLG0104" H 4750 3825 50  0001 C CNN
-F 1 "PWR_FLAG" H 4750 3923 50  0000 C CNN
-F 2 "" H 4750 3750 50  0001 C CNN
-F 3 "~" H 4750 3750 50  0001 C CNN
-	1    4750 3750
-	-1   0    0    1
+L power:GND #PWR0104
+U 1 1 5C8D3109
+P 4750 3650
+F 0 "#PWR0104" H 4750 3400 50  0001 C CNN
+F 1 "GND" H 4755 3477 50  0000 C CNN
+F 2 "" H 4750 3650 50  0001 C CNN
+F 3 "" H 4750 3650 50  0001 C CNN
+	1    4750 3650
+	1    0    0    -1
 $EndComp
-Wire Wire Line
-	4750 3750 4750 3650
 Connection ~ 4750 3650
 Wire Wire Line
 	4750 3650 5000 3650
+$Comp
+L power:+5V #PWR0115
+U 1 1 5C909EB9
+P 6250 3250
+F 0 "#PWR0115" H 6250 3100 50  0001 C CNN
+F 1 "+5V" H 6265 3423 50  0000 C CNN
+F 2 "" H 6250 3250 50  0001 C CNN
+F 3 "" H 6250 3250 50  0001 C CNN
+	1    6250 3250
+	1    0    0    -1
+$EndComp
+Connection ~ 6250 3250
 Wire Wire Line
-	4750 3150 4750 3250
-Connection ~ 5000 3250
-Wire Wire Line
-	4600 3250 4750 3250
-Text HLabel 6350 3250 2    50   Input ~ 0
-+5
-Connection ~ 4750 3250
-Wire Wire Line
-	4750 3250 5000 3250
+	6250 3250 6350 3250
 $EndSCHEMATC

Commit message: Izlabots majas darbs Nr.2
Changed lines of the file:
@@
 EESchema Schematic File Version 4
+LIBS:PWR_Supply-cache
 EELAYER 26 0
 EELAYER END
@@
 	1    0    0    -1
 $EndComp
-Wire Wire Line
-	6050 3250 6250 3250
 Connection ~ 6050 3250
 Connection ~ 5000 3650
 Connection ~ 5000 3250
-Text HLabel 6350 3250 2    50   Input ~ 0
+Text HLabel 6350 3250 2    50   Output ~ 0
 +5
 Wire Wire Line
@@
 $Comp
 L power:VCC #PWR0103
-U 1 1 5C8D30D8
+U 1 1 5C8F8141
 P 4750 3250
 F 0 "#PWR0103" H 4750 3100 50  0001 C CNN
@@
 $Comp
 L power:GND #PWR0104
-U 1 1 5C8D3109
+U 1 1 5C8F819B
 P 4750 3650
 F 0 "#PWR0104" H 4750 3400 50  0001 C CNN
@@
 Wire Wire Line
 	4750 3650 5000 3650
+Wire Wire Line
+	6250 3250 6350 3250
+Wire Wire Line
+	6050 3250 6250 3250
+Connection ~ 6250 3250
 $Comp
 L power:+5V #PWR0115
@@
 	1    0    0    -1
 $EndComp
-Connection ~ 6250 3250
-Wire Wire Line
-	6250 3250 6350 3250
 $EndSCHEMATC

Commit message: Izlabots majas darbs Nr.2
Parts:
- U1: value L7805 -> LM7805
Changed lines of the file:
@@
 P 5500 3250
 F 0 "U1" H 5500 3492 50  0000 C CNN
-F 1 "L7805" H 5500 3401 50  0000 C CNN
+F 1 "LM7805" H 5500 3401 50  0000 C CNN
 F 2 "" H 5525 3100 50  0001 L CIN
-F 3 "http://www.st.com/content/ccc/resource/technical/document/datasheet/41/4f/b3/b0/12/d4/47/88/CD00000444.pdf/files/CD00000444.pdf/jcr:content/translations/en.CD00000444.pdf" H 5500 3200 50  0001 C CNN
+F 3 "http://pdf1.alldatasheet.com/datasheet-pdf/view/82833/FAIRCHILD/LM7805.html" H 5500 3200 50  0001 C CNN
 	1    5500 3250
 	1    0    0    -1
