File: PWR_Supply/9V_DC.sch (KiCad schematic (older format))
At the start: 3 parts, among them U3 L7809

Commit message: Izlabots Majas Darbs Nr.2
Connections:
- net +9 renamed +9V
Changed lines of the file:
@@
 EESchema Schematic File Version 4
-LIBS:PWR_Supply-cache
 EELAYER 26 0
 EELAYER END
@@
 Wire Wire Line
 	5400 3400 4800 3400
-Wire Wire Line
-	4800 3000 4600 3000
 Connection ~ 4800 3000
 Connection ~ 4800 3400
@@
 +9
 Connection ~ 5950 3000
+Wire Wire Line
+	5950 3000 6150 3000
+Wire Wire Line
+	4450 3000 4600 3000
+Wire Wire Line
+	4450 3400 4600 3400
 $Comp
-L power:PWR_FLAG #FLG0105
-U 1 1 5C8E3782
-P 4600 2900
-F 0 "#FLG0105" H 4600 2975 50  0001 C CNN
-F 1 "PWR_FLAG" H 4600 3074 50  0000 C CNN
-F 2 "" H 4600 2900 50  0001 C CNN
-F 3 "~" H 4600 2900 50  0001 C CNN
-	1    4600 2900
+L power:GND #PWR0105
+U 1 1 5C8D3160
+P 4600 3400
+F 0 "#PWR0105" H 4600 3150 50  0001 C CNN
+F 1 "GND" H 4605 3227 50  0000 C CNN
+F 2 "" H 4600 3400 50  0001 C CNN
+F 3 "" H 4600 3400 50  0001 C CNN
+	1    4600 3400
 	1    0    0    -1
 $EndComp
-$Comp
-L power:PWR_FLAG #FLG0106
-U 1 1 5C8E37AD
-P 4600 3500
-F 0 "#FLG0106" H 4600 3575 50  0001 C CNN
-F 1 "PWR_FLAG" H 4600 3673 50  0000 C CNN
-F 2 "" H 4600 3500 50  0001 C CNN
-F 3 "~" H 4600 3500 50  0001 C CNN
-	1    4600 3500
-	-1   0    0    1
-$EndComp
-Wire Wire Line
-	4600 3000 4600 2900
-Connection ~ 4600 3000
-Wire Wire Line
-	4600 3000 4450 3000
-Wire Wire Line
-	4450 3400 4600 3400
-Wire Wire Line
-	4600 3500 4600 3400
 Connection ~ 4600 3400
 Wire Wire Line
 	4600 3400 4800 3400
+$Comp
+L power:VCC #PWR0106
+U 1 1 5C8D3191
+P 4600 3000
+F 0 "#PWR0106" H 4600 2850 50  0001 C CNN
+F 1 "VCC" H 4617 3173 50  0000 C CNN
+F 2 "" H 4600 3000 50  0001 C CNN
+F 3 "" H 4600 3000 50  0001 C CNN
+	1    4600 3000
+	1    0    0    -1
+$EndComp
+Connection ~ 4600 3000
 Wire Wire Line
-	5950 3000 6300 3000
+	4600 3000 4800 3000
+$Comp
+L power:+9V #PWR0116
+U 1 1 5C909F0F
+P 6150 3000
+F 0 "#PWR0116" H 6150 2850 50  0001 C CNN
+F 1 "+9V" H 6165 3173 50  0000 C CNN
+F 2 "" H 6150 3000 50  0001 C CNN
+F 3 "" H 6150 3000 50  0001 C CNN
+	1    6150 3000
+	1    0    0    -1
+$EndComp
+Connection ~ 6150 3000
+Wire Wire Line
+	6150 3000 6300 3000
 $EndSCHEMATC

Commit message: Izlabots majas darbs Nr.2
Changed lines of the file:
@@
 EESchema Schematic File Version 4
+LIBS:PWR_Supply-cache
 EELAYER 26 0
 EELAYER END
@@
 Text HLabel 4450 3400 0    50   Input ~ 0
 GND
-Text HLabel 6300 3000 2    50   Input ~ 0
+Text HLabel 6300 3000 2    50   Output ~ 0
 +9
 Connection ~ 5950 3000

Commit message: Izlabots majas darbs Nr.2
Parts:
- U3: value L7809 -> LM7809
Changed lines of the file:
@@
 P 5400 3000
 F 0 "U3" H 5400 3242 50  0000 C CNN
-F 1 "L7809" H 5400 3151 50  0000 C CNN
+F 1 "LM7809" H 5400 3151 50  0000 C CNN
 F 2 "" H 5425 2850 50  0001 L CIN
-F 3 "http://www.st.com/content/ccc/resource/technical/document/datasheet/41/4f/b3/b0/12/d4/47/88/CD00000444.pdf/files/CD00000444.pdf/jcr:content/translations/en.CD00000444.pdf" H 5400 2950 50  0001 C CNN
+F 3 "http://pdf1.alldatasheet.com/datasheet-pdf/view/33410/UTC/LM7809.html" H 5400 2950 50  0001 C CNN
 	1    5400 3000
 	1    0    0    -1
